File: pongCard/pongCard.kicad_pcb (KiCad board)
At the start: 2 copper layers, 83 x 54 mm, 26 parts, among them J1 USB_B_Micro, J2 Conn_02x04_Odd_Even, J3 Conn_02x04_Odd_Even, U1 ESP-01v090, U2 HT75xx-1-SOT89, U3 ESP-12E

Commit message: V3: Battery Step up
Parts:
- added BT1: AAA, pongCard:BatteryHolder_AAA_MYOUNG, B.Cu at (73.8, 65.1)
- added BT2: AAA, pongCard:BatteryHolder_AAA_MYOUNG, B.Cu at (129.9, 110.6)
- added C8: 100u, Capacitor_SMD:C_1206_3216Metric_Pad1.33x1.80mm_HandSolder, F.Cu at (76.3, 69.1)
- added C9: 100n, Capacitor_SMD:C_0603_1608Metric_Pad1.08x0.95mm_HandSolder, F.Cu at (75.6, 71.4)
- added D1: 1N5819, Diode_SMD:D_SOD-123, F.Cu at (85.7, 83.0)
- added L1: 47µ, Inductor_SMD:L_1210_3225Metric_Pad1.42x2.65mm_HandSolder, F.Cu at (75.1, 81.1)
- added SW1: SW_SPDT_COM, pongCard:SW_SPDT_PCM12_COM, F.Cu at (79.5, 63.7)
- added U4: QX2303L33E, Package_TO_SOT_SMD:SOT-89-3_Handsoldering, F.Cu at (81.2, 81.3)
- U2: footprint Package_TO_SOT_SMD:SOT-89-3 -> Package_TO_SOT_SMD:SOT-89-3_Handsoldering
- moved J1 7.15 mm to (87.8, 64.1)
- moved U2 5.34 mm to (83.2, 74.2)
- moved C3 4.25 mm to (81.9, 70.4)
- moved C4 2.34 mm to (81.2, 68.4)
- moved C2 0.38 mm to (102.9, 88.2)
- moved C1 0.15 mm to (103.0, 90.2)
Routing:
- net Net-(BT1--): track 0.00 -> 57.0 mm
- net Net-(SW1-B): track 0.00 -> 17.0 mm
- net GND: track 33.2 -> 48.8 mm, vias 40 -> 50
- net Net-(J1-VBUS): track 16.3 -> 3.66 mm
- net Net-(D1-A): track 0.00 -> 11.5 mm
- net Net-(BT1-+): track 0.00 -> 4.25 mm
- net Net-(JP2-A): track 146.8 -> 148.7 mm
